File: hardware/sret.kicad_pcb (KiCad board)
At the start: 4 copper layers, 90 x 90 mm, 105 parts, among them J1 RJ45-TRANSFO, P1 USB0, P10 CONN_02X04, P11 USB1, P12 CONN_02X01, P13 CONN_02X01, P14 CONN_02X01, P2 CONN_02X01, P3 CONN_02X01, P4 CONN_02X01, P5 CONN_02X01, P6 CONN_01X06, P7 CONN_01X06, P8 CONN_01X06, P9 CONN_01X06, SW1 DFU, SW2 RESET, U1 LPC4330, U2 DRTR5V0U2SR, U3 W25Q80BV, U4 LAN8742A, U5 MAX3051, U6 MAX3051, U7 TC1262, U8 RS-485/IEBus, X1 CRYSTAL_SMD, X2 CRYSTAL_SMD, Y1 RTC

Commit message: more traces
Parts:
- P1, P11: moved to B.Cu
- moved R21 73.3 mm to (176.0, 70.7), turned to 270 degrees
- moved P5 72.8 mm to (176.9, 55.9), turned to 0 degrees
- moved R25 70.9 mm to (176.0, 68.0), turned to 270 degrees
- moved P9 62.5 mm to (179.4, 59.7)
- moved C19 39.6 mm to (236.3, 78.1), turned to 0 degrees
- moved C30 37.6 mm to (196.4, 85.3), turned to 225 degrees
- moved P13 24.0 mm to (176.2, 45.8)
- moved R13 23.7 mm to (174.3, 94.2), turned to 0 degrees
- moved U6 18.6 mm to (175.7, 39.0)
- moved R36 13.2 mm to (199.9, 33.6)
- moved R6 12.3 mm to (169.4, 85.9), turned to 270 degrees
- moved R16 11.3 mm to (174.3, 98.8)
- moved U2 10.8 mm to (172.0, 88.7), turned to 0 degrees
- moved P12 10.7 mm to (194.7, 43.4), turned to 180 degrees
- moved R35 9.32 mm to (202.3, 33.6), turned to 270 degrees
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Connections:
- SGPIO1 pad 12: /SGPIO11 -> /SGPIO11/USB1_VBUS
Routing:
- net /RESET#: track 0.00 -> 168.4 mm, vias 0 -> 5
- net GND: track 0.00 -> 162.7 mm, vias 0 -> 26
- net VCC: track 0.00 -> 157.2 mm, vias 0 -> 19
- net /GPIO4: track 0.00 -> 97.0 mm, vias 0 -> 2
- net /GPIO16: track 0.00 -> 89.4 mm, vias 0 -> 3
- net /CAN1_RXD: track 0.00 -> 81.9 mm, vias 0 -> 4
- net /GP_CLKIN: track 0.00 -> 81.6 mm, vias 0 -> 4
- net /BOOT0/SSPO_MISO/EMC_A6: track 0.00 -> 78.8 mm, vias 0 -> 1
- net /ADC0: track 0.00 -> 78.5 mm, vias 0 -> 4
- net /BOOT1/SSGPIO6/SSPO_MOSI/EMC_A7: track 0.00 -> 76.6 mm, vias 0 -> 3
- net /GPIO2: track 0.00 -> 74.7 mm, vias 0 -> 2
- net /ADC6: track 0.00 -> 74.0 mm, vias 0 -> 4
- net /SD_DATA0/EMC_D1: track 0.00 -> 73.1 mm, vias 0 -> 2
- net /EMC_D2: track 0.00 -> 72.8 mm, vias 0 -> 2
- net /ADC1: track 0.00 -> 71.7 mm, vias 0 -> 2
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- added copper zone on B.Cu, net /5V
