File: hardware/sret.sch (KiCad schematic (older format))
At the start: 109 parts, among them CON1 SD_Card, J1 RJ45-TRANSFO, P1 USB0, P10 CONN_02X04, P11 USB1, P12 CONN_02X01, P13 CONN_02X01, P14 CONN_02X01, P2 CONN_02X01, P3 CONN_02X01, P4 CONN_02X01, P5 CONN_02X01, P6 CONN_01X06, P7 CONN_01X06, P8 CONN_01X06, P9 CONN_01X06, SW1 DFU, SW2 RESET, U1 LPC4330, U2 DRTR5V0U2SR, U3 W25Q80BV, U4 LAN8742A, U5 MAX3051, U6 MAX3051, U7 TC1262, U8 RS-485/IEBus, X1 CRYSTAL_SMD, X2 CRYSTAL_SMD, Y1 RTC

Commit message: pcb routing started
Parts:
- P1, P11: footprint Connect:USB_Micro-B -> Connect:USB_Micro-B_circle

Commit message: 2nd version pcb
Parts:
- removed CON1: SD_Card, Connect:SD_Card_Receptacle, symbol SD_Card
- removed R11, R8, R9: 1k5, Resistors_SMD:R_0603_HandSoldering, symbol R
- C1, C10, C11, C12, C13, C14, C15, C16, C17, C18, C19, C2, C20, C21, C22, C23, C24, C25, C26, C27, C28, C29, C3, C30, C31, C32, C4, C5, C6, C7, C8, C9: footprint Capacitors_SMD:C_0603_HandSoldering -> Capacitors_SMD:C_0603
- R1, R10, R12, R13, R14, R15, R16, R17, R18, R19, R2, R20, R21, R22, R23, R24, R25, R26, R27, R28, R29, R3, R30, R31, R32, R33, R34, R35, R36, R4, R5, R6, R7: footprint Resistors_SMD:R_0603_HandSoldering -> Resistors_SMD:R_0603
Connections:
- net SD_CLK: now also P9.2 (P2)
- no-connect marks 15 -> 9
Other:
- note removed: "Not sure if SD lines need pull-up/down resistors."

Commit message: update pcb
Connections:
- net CANL_0: no longer GPIO1.22 (P22)
- net CANL_1: now also GPIO1.22 (P22)

Commit message: more traces
Connections:
- net SGPIO11 is gone; now on net SGPIO11/USB1_VBUS: SGPIO1.12 (P12)
Changed lines of the file:
@@
 Text Label 7500 3750 0    60   ~ 0
 SGPIO11/USB1_VBUS
-Text Label 15000 8350 0    60   ~ 0
-SGPIO11
 Text Label 7500 3650 0    60   ~ 0
 SCL
@@
 Wire Wire Line
 	16100 2850 15800 2850
+Text Label 15000 8350 0    60   ~ 0
+SGPIO11/USB1_VBUS
 $EndSCHEMATC
